File: Test/Test.kicad_sch (KiCad schematic)
At the start: 12 parts, among them IC1 E-L9637D

Commit message: Hadley's changes
13/09/2026

Co-Authored-By: stupid-crackers <326826861+stupid-crackers@users.noreply.github.com>
Parts:
- removed V1: VPWL, symbol Simulation_SPICE:VPWL
- added C3, C4: 100n, Capacitor_THT:C_Rect_L7.0mm_W2.5mm_P5.00mm, symbol uc_components:UC_C
- added D3: 1N4148, Diode_THT:D_DO-35_SOD27_P7.62mm_Horizontal, symbol Diode:1N4148
- added J1, J3: Conn_01x02, Package_DFN_QFN:QFN-20-1EP_5x5mm_P0.65mm_EP3.35x3.35mm, symbol Connector_Generic:Conn_01x02
- added J4: Conn_01x10, Package_DFN_QFN:QFN-20-1EP_5x5mm_P0.65mm_EP3.35x3.35mm, symbol Connector_Generic:Conn_01x10
- added J5: Conn_01x04, Package_DFN_QFN:QFN-20-1EP_5x5mm_P0.65mm_EP3.35x3.35mm, symbol Connector_Generic:Conn_01x04
- added SW1: RotaryEncoder_Switch, Package_DFN_QFN:QFN-28-1EP_6x6mm_P0.65mm_EP4.25x4.25mm, symbol Device:RotaryEncoder_Switch
- D1: value 1N5824 -> MBR560S
Connections:
- net +12V: now also C3.1, D3.2 (A); no longer IC1.7 (VS)
- net +5V: now also A1.39 (VSYS), J5.1 (Pin_1); no longer IC1.3 (VCC)
- net GND: now also J2.4 (Chassis_Ground); no longer A1.13 (GND), A1.18 (GND), A1.23 (GND), A1.28 (GND), A1.3 (GND), A1.38 (GND), A1.8 (GND), C1.2, D1.A, IC1.5 (GND), IC1.8 (LI), VR1.5 (~{ON}/OFF)
- net GPI02: now reaches IC1.2 (LO)
- net GPI02: now also A1.4 (GPIO2)
- net at F1.1: now also J2.16 (Battery_Power)
- net L line: now reaches J2.15 (ISO_9141-2_LOW)
- net L line: now also IC1.8 (LI)
- net GNDS: now reaches J2.5 (Signal_Ground)
- net GNDS: now also A1.13 (GND), A1.18 (GND), A1.23 (GND), A1.28 (GND), A1.3 (GND), A1.38 (GND), A1.8 (GND), C1.2, D1.A, IC1.5 (GND), VR1.5 (~{ON}/OFF), C3.2, C4.2, J1.2 (Pin_2), J3.2 (Pin_2), J4.10 (Pin_10), J4.2 (Pin_2), J5.2 (Pin_2), SW1.S2
- net GPIO16: now reaches A1.21 (GPIO16)
- net GPIO16: now also J1.1 (Pin_1)
- net GPIO17: now reaches A1.22 (GPIO17)
- net GPIO17: now also J3.1 (Pin_1)
- net SCA: now reaches A1.24 (GPIO18)
- net SCA: now also J4.4 (Pin_4)
- net SCL: now reaches A1.25 (GPIO19)
- net SCL: now also J4.3 (Pin_3)
- net SDA: now reaches A1.26 (GPIO20)
- net SDA: now also J5.3 (Pin_3)
- net SCL2: now reaches A1.27 (GPIO21)
- net SCL2: now also J5.4 (Pin_4)
- net +3.3V: now reaches A1.36 (3V3)
- net +3.3V: now also IC1.3 (VCC), C4.1, J4.1 (Pin_1)
- net GPIO6: now reaches A1.9 (GPIO6)
- net GPIO6: now also SW1.S1
- new net: D3.1 (K), IC1.7 (VS)
- new net ADO: J4.7 (Pin_7)
- new net ECL: J4.6 (Pin_6)
- new net EDA: J4.5 (Pin_5)
- new net FCS: J4.9 (Pin_9)
- new net INT: J4.8 (Pin_8)
- no-connect marks 47 -> 32
Other:
- note added: "9 Axis Accelerometer, GY-9250"
- note added: "Start Stop Lap Switches"
- note added: "Use solder connectors, Use as a button for start stop lap"
- moved on the sheet: A1, D2, F1, IC1, J2, R1
