File: Test/Test.kicad_pcb (KiCad board)
At the start: 2 copper layers, 6 parts

Commit message: Final pcb
PCB routed 15/09/2026

Co-Authored-By: G7Connoisseur <326818386+G7Connoisseur@users.noreply.github.com>
Co-Authored-By: stupid-crackers <326826861+stupid-crackers@users.noreply.github.com>
Parts:
- removed A1: RaspberryPi_Pico_W, Module:RaspberryPi_Pico_W_SMD_HandSolder
- removed C1: 220u, Capacitor_THT:C_Rect_L7.0mm_W2.5mm_P5.00mm
- removed C2: 680u, Capacitor_THT:C_Rect_L7.0mm_W2.5mm_P5.00mm
- removed L1: l=33u, Inductor_THT:L_Axial_L6.6mm_D2.7mm_P2.54mm_Vertical_Vishay_IM-2
- removed VR1: LM2596S-5.0, OBD2:TO170P1524X483-6N
- added C3: 100n, Capacitor_THT:C_Rect_L4.6mm_W3.0mm_P2.50mm_MKS02_FKP02, F.Cu at (155.5, 56.5)
- added C4: 100n, Capacitor_THT:C_Rect_L4.6mm_W3.0mm_P2.50mm_MKS02_FKP02, F.Cu at (143.5, 62.5)
- added C5: 100u, Capacitor_THT:CP_Radial_D6.3mm_P2.50mm, F.Cu at (189.6, 102.2)
- added C6: 1000u, Capacitor_THT:CP_Radial_D12.5mm_P5.00mm, F.Cu at (180.1, 95.7)
- added CR1: E-L9637D, Package_SO:SO-8_3.9x4.9mm_P1.27mm, F.Cu at (149.0, 59.8)
- added D2: 1.5KE24A, Diode_THT:D_DO-201_P5.08mm_Vertical_AnodeUp, F.Cu at (193.1, 78.1)
- added D3: 1N4148, Diode_THT:D_DO-201_P5.08mm_Vertical_AnodeUp, F.Cu at (165.5, 55.8)
- added D4: MBR360, Diode_THT:D_DO-201_P5.08mm_Vertical_AnodeUp, F.Cu at (190.6, 94.6)
- added F1: Fuse, Fuse:Fuseholder_Clip-5x20mm_Schurter_CQM_Inline_P20.60x5.00mm_D1.00mm_Horizontal, F.Cu at (187.0, 51.7)
- added J1: Conn_01x02, Connector_PinHeader_2.54mm:PinHeader_1x02_P2.54mm_Vertical, F.Cu at (155.0, 121.5)
- added J2: Conn_01x20, Connector_PinHeader_2.54mm:PinHeader_1x20_P2.54mm_Vertical, F.Cu at (134.5, 80.6)
- added J3: Conn_01x02, Connector_PinHeader_2.54mm:PinHeader_1x02_P2.54mm_Vertical, F.Cu at (145.2, 121.5)
- added J4: Conn_01x10, Connector_PinSocket_2.54mm:PinSocket_1x10_P2.54mm_Vertical, F.Cu at (139.0, 89.0)
- added J5: Conn_01x04, Connector_PinHeader_2.54mm:PinHeader_1x04_P2.54mm_Vertical, F.Cu at (139.0, 123.0)
- added J6: Conn_01x05, Connector_PinHeader_2.54mm:PinHeader_1x05_P2.54mm_Vertical, F.Cu at (193.5, 51.5)
- added J7: Conn_01x20, Connector_PinHeader_2.54mm:PinHeader_1x20_P2.54mm_Vertical, F.Cu at (115.5, 80.6)
- added L2: 100u, Inductor_THT:L_Toroid_Horizontal_D24.1mm_P21.80mm_Bourns_2200, F.Cu at (149.2, 100.5)
- added R1: 510, Resistor_THT:R_Axial_DIN0207_L6.3mm_D2.5mm_P7.62mm_Horizontal, F.Cu at (163.5, 63.8)
- added R2: 10k, Resistor_THT:R_Axial_DIN0207_L6.3mm_D2.5mm_P7.62mm_Horizontal, F.Cu at (105.5, 70.3)
- added R3: 10k, Resistor_THT:R_Axial_DIN0207_L6.3mm_D2.5mm_P7.62mm_Horizontal, F.Cu at (150.3, 125.0)
- added R4: 10k, Resistor_THT:R_Axial_DIN0207_L6.3mm_D2.5mm_P7.62mm_Horizontal, F.Cu at (116.5, 62.7)
- added R5: 10k, Resistor_THT:R_Axial_DIN0207_L6.3mm_D2.5mm_P7.62mm_Horizontal, F.Cu at (110.5, 70.3)
- added R6: 10k, Resistor_THT:R_Axial_DIN0207_L6.3mm_D2.5mm_P7.62mm_Horizontal, F.Cu at (153.2, 125.0)
- added S1: PEC11R-4220F-S0024, KiCad online models:XDCR_PEC11R-4220F-S0024, F.Cu at (114.5, 54.0)
- added U1: LM2576T-5, Package_TO_SOT_THT:TO-220-5_Vertical, F.Cu at (182.6, 110.9)
- D1: value 1N5824 -> 1N5408; footprint OBD2:DIOAD1898W129L762D1143 -> Diode_THT:D_DO-201_P5.08mm_Vertical_AnodeUp
- moved D1 84.2 mm to (193.5, 71.4)
Routing:
- net +3.3V: track 0.00 -> 147.7 mm
- net +12V: track 2.64 -> 117.8 mm
- net +5V: track 0.00 -> 107.8 mm
- net /GPIO6: track 0.00 -> 76.1 mm
- net /GPIO8: track 0.00 -> 63.5 mm
- net /GPIO7: track 0.00 -> 60.6 mm
- net Net-(D4-K): track 0.00 -> 55.9 mm
- net /K_Line: track 0.00 -> 51.3 mm
- net /GPIO1: track 0.00 -> 47.3 mm
- net /L_Line: track 0.00 -> 47.0 mm, vias 0 -> 1
- net /GPIO0: track 0.00 -> 40.2 mm
- net /SCL: track 0.00 -> 21.2 mm
- net /SCA: track 0.00 -> 21.2 mm
- net Net-(CR1-VS): track 0.00 -> 17.1 mm
- net /GPIO17: track 0.00 -> 13.1 mm
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- added copper zone on B.Cu, net GND
Other:
- board outline added: 95 x 95 mm
- board text added: "BUCK CONVERTER STEP DOWN"
- board text added: "CIRCUIT INPUT AND PROTECTION"
- board text added: "ENCODER/SWITCH"
- board text added: "GROUP 40."
- board text added: "HADLEY LUMB, CODY SODEN, HAMISH MCKINLAY"
- board text added: "TRANCEIVER INPUT OUTPUT"
