File: Test/_restore_backup_2026-09-14T21-57-21-956/Test.kicad_sch (KiCad schematic)
At the start: 27 parts, among them J1 Conn_01x02, J2 Conn_01x20, J3 Conn_01x02, J4 Conn_01x10, J5 Conn_01x04, J6 Conn_01x05, J7 Conn_01x20, U1 LM2576T-5

Commit message: Final pcb
PCB routed 15/09/2026

Co-Authored-By: G7Connoisseur <326818386+G7Connoisseur@users.noreply.github.com>
Co-Authored-By: stupid-crackers <326826861+stupid-crackers@users.noreply.github.com>
Parts:
- removed J2, J7: Conn_01x20, Connector_PinHeader_2.54mm:PinHeader_1x20_P2.54mm_Vertical, symbol Connector_Generic:Conn_01x20
- removed S1: PEC11R-4220F-S0024, KiCad online models:XDCR_PEC11R-4220F-S0024, symbol PEC11R-4220F-S0024:PEC11R-4220F-S0024
- C3, C4: footprint Capacitor_THT:C_Rect_L4.6mm_W3.0mm_P2.50mm_MKS02_FKP02 -> Capacitor_THT:C_Rect_L7.0mm_W2.5mm_P5.00mm
- C5: footprint Capacitor_THT:CP_Radial_D6.3mm_P2.50mm -> Capacitor_THT:C_Rect_L7.0mm_W2.5mm_P5.00mm
- C6: footprint Capacitor_THT:CP_Radial_D12.5mm_P5.00mm -> Capacitor_THT:C_Rect_L7.0mm_W2.5mm_P5.00mm
- CR1: footprint Package_SO:SO-8_3.9x4.9mm_P1.27mm -> footprints:SO-8_STM
Connections:
- net +12V: now also C3.1
- net +3.3V: now also R2.1, R5.1; no longer R2.2, R5.2
- net GPIO7: now also R5.2; no longer R5.1
- net GPIO8: now also R2.2; no longer R2.1
- net at CR1.7 (VS), D3.1 (K): no longer C3.1
- no-connect marks 42 -> 24
Other:
- moved on the sheet: C3, C5, C6, D1, D2, D3, D4, F1, J1, J3, J4, J5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
